File: RAMPS-FD/Extra_Mosfets.sch (KiCad schematic (older format))
At the start: 12 parts, among them P901 D12, P902 D2, Q901 DMN2075U, Q902 DMN2075U

Commit message: Changed fuse holders to Keystone 3568; specificy HCT instead of ACT logic
Parts:
- D901, D902: symbol LED -> LED-RESCUE-RAMPS-FD
- D903, D904: symbol DIODE -> D
Connections:
- net +12P: now also D903.1 (K), D904.1 (K); no longer D903.2 (K), D904.2 (K)
- net P_FET5: now also D903.2 (A); no longer D903.1 (A)
- net P_FET6: now also D904.2 (A); no longer D904.1 (A)
Changed lines of the file:
@@
 Connection ~ 3500 2050
 Wire Wire Line
-	3500 1700 3500 2200
+	3500 1650 3500 2200
 Wire Wire Line
 	3000 1000 3000 1150
@@
 	3900 1850 3900 1000
 Wire Wire Line
-	3500 850  3500 1300
+	3500 850  3500 1350
 $Comp
 L MOSFET_N Q901
@@
 $EndComp
 $Comp
-L DIODE D903
+L D D903
 U 1 1 523E6004
 P 3500 1500
@@
 F 3 "" H 3500 1500 60  0001 C CNN
 	1    3500 1500
-	0    -1   -1   0
+	0    1    1    0
 $EndComp
 $Comp
-L LED D901
+L LED-RESCUE-RAMPS-FD D901
 U 1 1 523E6017
 P 3000 1800
@@
 Connection ~ 3500 5250
 Wire Wire Line
-	3500 4900 3500 5400
+	3500 4850 3500 5400
 Wire Wire Line
 	3000 4200 3000 4350
@@
 	3900 5050 3900 4200
 Wire Wire Line
-	3500 4050 3500 4500
+	3500 4050 3500 4550
 $Comp
 L MOSFET_N Q902
@@
 $EndComp
 $Comp
-L DIODE D904
+L D D904
 U 1 1 523E66B7
 P 3500 4700
@@
 F 3 "" H 3500 4700 60  0001 C CNN
 	1    3500 4700
-	0    -1   -1   0
+	0    1    1    0
 $EndComp
 $Comp
-L LED D902
+L LED-RESCUE-RAMPS-FD D902
 U 1 1 523E66BD
 P 3000 5000
