File: RAMPS-FD/con_misc.sch (KiCad schematic (older format))
At the start: 17 parts, among them K201 S1, K202 S2, K203 S3, K204 S4, P1 SERIAL1, P2 I2C-1, P211 I2C-0, P213 AUX-4, P214 AUX-2, P215 AUX-3, P216 SERIAL0, U601 24C512

Commit message: Changed fuse holders to Keystone 3568; specificy HCT instead of ACT logic
Parts:
- K201, K202, K203, K204: footprint pin_array:PIN_ARRAY_3X1 -> Pin_Headers:Pin_Header_Straight_1x03
- P1, P216: footprint w_pin_strip:pin_strip_6 -> Pin_Headers:Pin_Header_Straight_1x06
- P2: footprint w_pin_strip:pin_strip_4 -> Pin_Headers:Pin_Header_Straight_1x04
- P211: footprint pin_array:PIN_ARRAY_4x1 -> Pin_Headers:Pin_Header_Straight_1x04
- P213: footprint w_pin_strip:pin_strip_18 -> Pin_Headers:Pin_Header_Straight_1x18
Changed lines of the file:
@@
 F 0 "P2" V 5750 4550 50  0000 C CNN
 F 1 "I2C-1" V 5850 4550 50  0000 C CNN
-F 2 "w_pin_strip:pin_strip_4" H 5800 4550 60  0001 C CNN
+F 2 "Pin_Headers:Pin_Header_Straight_1x04" H 5800 4550 60  0001 C CNN
 F 3 "" H 5800 4550 60  0001 C CNN
 	1    5800 4550
@@
 F 0 "P1" V 2750 3050 60  0000 C CNN
 F 1 "SERIAL1" V 2850 3050 60  0000 C CNN
-F 2 "w_pin_strip:pin_strip_6" H 2800 3050 60  0001 C CNN
+F 2 "Pin_Headers:Pin_Header_Straight_1x06" H 2800 3050 60  0001 C CNN
 F 3 "" H 2800 3050 60  0001 C CNN
 	1    2800 3050
@@
 F 0 "P216" V 2750 1800 60  0000 C CNN
 F 1 "SERIAL0" V 2850 1800 60  0000 C CNN
-F 2 "w_pin_strip:pin_strip_6" H 2800 1800 60  0001 C CNN
+F 2 "Pin_Headers:Pin_Header_Straight_1x06" H 2800 1800 60  0001 C CNN
 F 3 "" H 2800 1800 60  0001 C CNN
 	1    2800 1800
@@
 F 0 "P213" V 9650 5575 60  0000 C CNN
 F 1 "AUX-4" V 9750 5575 60  0000 C CNN
-F 2 "w_pin_strip:pin_strip_18" H 9700 5575 60  0001 C CNN
+F 2 "Pin_Headers:Pin_Header_Straight_1x18" H 9700 5575 60  0001 C CNN
 F 3 "" H 9700 5575 60  0001 C CNN
 	1    9700 5575
@@
 F 0 "K204" V 2000 6650 50  0000 C CNN
 F 1 "S4" V 2100 6650 40  0000 C CNN
-F 2 "pin_array:PIN_ARRAY_3X1" H 2050 6650 60  0001 C CNN
+F 2 "Pin_Headers:Pin_Header_Straight_1x03" H 2050 6650 60  0001 C CNN
 F 3 "" H 2050 6650 60  0001 C CNN
 	1    2050 6650
@@
 F 0 "K203" V 2000 5900 50  0000 C CNN
 F 1 "S3" V 2100 5900 40  0000 C CNN
-F 2 "pin_array:PIN_ARRAY_3X1" H 2050 5900 60  0001 C CNN
+F 2 "Pin_Headers:Pin_Header_Straight_1x03" H 2050 5900 60  0001 C CNN
 F 3 "" H 2050 5900 60  0001 C CNN
 	1    2050 5900
@@
 F 0 "K202" V 2000 5250 50  0000 C CNN
 F 1 "S2" V 2100 5250 40  0000 C CNN
-F 2 "pin_array:PIN_ARRAY_3X1" H 2050 5250 60  0001 C CNN
+F 2 "Pin_Headers:Pin_Header_Straight_1x03" H 2050 5250 60  0001 C CNN
 F 3 "" H 2050 5250 60  0001 C CNN
 	1    2050 5250
@@
 F 0 "K201" V 2000 4500 50  0000 C CNN
 F 1 "S1" V 2100 4500 40  0000 C CNN
-F 2 "pin_array:PIN_ARRAY_3X1" H 2050 4500 60  0001 C CNN
+F 2 "Pin_Headers:Pin_Header_Straight_1x03" H 2050 4500 60  0001 C CNN
 F 3 "" H 2050 4500 60  0001 C CNN
 	1    2050 4500
@@
 F 0 "P211" V 5750 2350 50  0000 C CNN
 F 1 "I2C-0" V 5850 2350 50  0000 C CNN
-F 2 "pin_array:PIN_ARRAY_4x1" H 5800 2350 60  0001 C CNN
+F 2 "Pin_Headers:Pin_Header_Straight_1x04" H 5800 2350 60  0001 C CNN
 F 3 "" H 5800 2350 60  0001 C CNN
 	1    5800 2350

Commit message: Fix 3d view; remove faulty ADC protection
Parts:
- K201, K202, K203, K204: footprint Pin_Headers:Pin_Header_Straight_1x03 -> Pin_Headers:Pin_Header_Straight_1x03_Pitch2.54mm
- P1, P216: footprint Pin_Headers:Pin_Header_Straight_1x06 -> Pin_Headers:Pin_Header_Straight_1x06_Pitch2.54mm
- P2, P211: footprint Pin_Headers:Pin_Header_Straight_1x04 -> Pin_Headers:Pin_Header_Straight_1x04_Pitch2.54mm
- P213: footprint Pin_Headers:Pin_Header_Straight_1x18 -> Pin_Headers:Pin_Header_Straight_1x18_Pitch2.54mm
Changed lines of the file:
@@
 F 0 "P2" V 5750 4550 50  0000 C CNN
 F 1 "I2C-1" V 5850 4550 50  0000 C CNN
-F 2 "Pin_Headers:Pin_Header_Straight_1x04" H 5800 4550 60  0001 C CNN
+F 2 "Pin_Headers:Pin_Header_Straight_1x04_Pitch2.54mm" H 5800 4550 60  0001 C CNN
 F 3 "" H 5800 4550 60  0001 C CNN
 	1    5800 4550
@@
 P 5250 4800
 AR Path="/523B601D" Ref="#PWR071"  Part="1"
-AR Path="/5176EFAC/523B601D" Ref="#PWR072"  Part="1"
-F 0 "#PWR072" H 5250 4800 30  0001 C CNN
+AR Path="/5176EFAC/523B601D" Ref="#PWR070"  Part="1"
+F 0 "#PWR070" H 5250 4800 30  0001 C CNN
 F 1 "GND" H 5250 4730 30  0001 C CNN
 F 2 "" H 5250 4800 60  0001 C CNN
@@
 SCL1
 $Comp
-L +V_LOGIC #PWR073
+L +V_LOGIC #PWR071
 U 1 1 523B601C
 P 4450 3800
-F 0 "#PWR073" H 4450 3770 30  0001 C CNN
+F 0 "#PWR071" H 4450 3770 30  0001 C CNN
 F 1 "+V_LOGIC" H 4450 3900 30  0000 C CNN
 F 2 "" H 4450 3800 60  0001 C CNN
@@
 P 1950 3600
 AR Path="/523B5AB9" Ref="#PWR073"  Part="1"
-AR Path="/5176EFAC/523B5AB9" Ref="#PWR074"  Part="1"
-F 0 "#PWR074" H 1950 3600 30  0001 C CNN
+AR Path="/5176EFAC/523B5AB9" Ref="#PWR072"  Part="1"
+F 0 "#PWR072" H 1950 3600 30  0001 C CNN
 F 1 "GND" H 1950 3530 30  0001 C CNN
 F 2 "" H 1950 3600 60  0001 C CNN
@@
 F 0 "P1" V 2750 3050 60  0000 C CNN
 F 1 "SERIAL1" V 2850 3050 60  0000 C CNN
-F 2 "Pin_Headers:Pin_Header_Straight_1x06" H 2800 3050 60  0001 C CNN
+F 2 "Pin_Headers:Pin_Header_Straight_1x06_Pitch2.54mm" H 2800 3050 60  0001 C CNN
 F 3 "" H 2800 3050 60  0001 C CNN
 	1    2800 3050
@@
 F 0 "P216" V 2750 1800 60  0000 C CNN
 F 1 "SERIAL0" V 2850 1800 60  0000 C CNN
-F 2 "Pin_Headers:Pin_Header_Straight_1x06" H 2800 1800 60  0001 C CNN
+F 2 "Pin_Headers:Pin_Header_Straight_1x06_Pitch2.54mm" H 2800 1800 60  0001 C CNN
 F 3 "" H 2800 1800 60  0001 C CNN
 	1    2800 1800
@@
 D51-MOSI
 $Comp
-L +V_LOGIC #PWR075
+L +V_LOGIC #PWR073
 U 1 1 517867DD
 P 7950 1750
-F 0 "#PWR075" H 7950 1720 30  0001 C CNN
+F 0 "#PWR073" H 7950 1720 30  0001 C CNN
 F 1 "+V_LOGIC" H 7950 1850 30  0000 C CNN
 F 2 "" H 7950 1750 60  0001 C CNN
@@
 $EndComp
 $Comp
-L +V_LOGIC #PWR076
+L +V_LOGIC #PWR074
 U 1 1 517867D0
 P 8250 6475
-F 0 "#PWR076" H 8250 6445 30  0001 C CNN
+F 0 "#PWR074" H 8250 6445 30  0001 C CNN
 F 1 "+V_LOGIC" H 8250 6575 30  0000 C CNN
 F 2 "" H 8250 6475 60  0001 C CNN
@@
 $EndComp
 $Comp
-L +V_LOGIC #PWR077
+L +V_LOGIC #PWR075
 U 1 1 517867C6
 P 4450 1600
-F 0 "#PWR077" H 4450 1570 30  0001 C CNN
+F 0 "#PWR075" H 4450 1570 30  0001 C CNN
 F 1 "+V_LOGIC" H 4450 1700 30  0000 C CNN
 F 2 "" H 4450 1600 60  0001 C CNN
@@
 P 9100 6425
 AR Path="/51084B2C" Ref="#PWR077"  Part="1"
-AR Path="/5176EFAC/51084B2C" Ref="#PWR078"  Part="1"
-F 0 "#PWR078" H 9100 6425 30  0001 C CNN
+AR Path="/5176EFAC/51084B2C" Ref="#PWR076"  Part="1"
+F 0 "#PWR076" H 9100 6425 30  0001 C CNN
 F 1 "GND" H 9100 6355 30  0001 C CNN
 F 2 "" H 9100 6425 60  0001 C CNN
@@
 F 0 "P213" V 9650 5575 60  0000 C CNN
 F 1 "AUX-4" V 9750 5575 60  0000 C CNN
-F 2 "Pin_Headers:Pin_Header_Straight_1x18" H 9700 5575 60  0001 C CNN
+F 2 "Pin_Headers:Pin_Header_Straight_1x18_Pitch2.54mm" H 9700 5575 60  0001 C CNN
 F 3 "" H 9700 5575 60  0001 C CNN
 	1    9700 5575
@@
 P 7550 3600
 AR Path="/5104884C" Ref="#PWR078"  Part="1"
-AR Path="/5176EFAC/5104884C" Ref="#PWR079"  Part="1"
-F 0 "#PWR079" H 7550 3600 30  0001 C CNN
+AR Path="/5176EFAC/5104884C" Ref="#PWR077"  Part="1"
+F 0 "#PWR077" H 7550 3600 30  0001 C CNN
 F 1 "GND" H 7550 3530 30  0001 C CNN
 F 2 "" H 7550 3600 60  0001 C CNN
@@
 P 10000 1900
 AR Path="/51048839" Ref="#PWR079"  Part="1"
-AR Path="/5176EFAC/51048839" Ref="#PWR080"  Part="1"
-F 0 "#PWR080" H 10000 1900 30  0001 C CNN
+AR Path="/5176EFAC/51048839" Ref="#PWR078"  Part="1"
+F 0 "#PWR078" H 10000 1900 30  0001 C CNN
 F 1 "GND" H 10000 1830 30  0001 C CNN
 F 2 "" H 10000 1900 60  0001 C CNN
@@
 P 1950 2350
 AR Path="/5104861F" Ref="#PWR080"  Part="1"
-AR Path="/5176EFAC/5104861F" Ref="#PWR081"  Part="1"
-F 0 "#PWR081" H 1950 2350 30  0001 C CNN
+AR Path="/5176EFAC/5104861F" Ref="#PWR079"  Part="1"
+F 0 "#PWR079" H 1950 2350 30  0001 C CNN
 F 1 "GND" H 1950 2280 30  0001 C CNN
 F 2 "" H 1950 2350 60  0001 C CNN
@@
 F 0 "K204" V 2000 6650 50  0000 C CNN
 F 1 "S4" V 2100 6650 40  0000 C CNN
-F 2 "Pin_Headers:Pin_Header_Straight_1x03" H 2050 6650 60  0001 C CNN
+F 2 "Pin_Headers:Pin_Header_Straight_1x03_Pitch2.54mm" H 2050 6650 60  0001 C CNN
 F 3 "" H 2050 6650 60  0001 C CNN
 	1    2050 6650
@@
 P 1550 6850
 AR Path="/51047C7E" Ref="#PWR081"  Part="1"
-AR Path="/5176EFAC/51047C7E" Ref="#PWR082"  Part="1"
-F 0 "#PWR082" H 1550 6850 30  0001 C CNN
+AR Path="/5176EFAC/51047C7E" Ref="#PWR080"  Part="1"
+F 0 "#PWR080" H 1550 6850 30  0001 C CNN
 F 1 "GND" H 1550 6780 30  0001 C CNN
 F 2 "" H 1550 6850 60  0001 C CNN
@@
 $EndComp
 $Comp
-L +5V #PWR083
+L +5V #PWR081
 U 1 1 51047C7D
 P 1550 6450
-F 0 "#PWR083" H 1550 6300 50  0001 C CNN
+F 0 "#PWR081" H 1550 6300 50  0001 C CNN
 F 1 "+5V" H 1550 6590 50  0000 C CNN
 F 2 "" H 1550 6450 50  0000 C CNN
@@
 SERVO3
 $Comp
-L +5V #PWR084
+L +5V #PWR082
 U 1 1 51047C7B
 P 1550 5700
-F 0 "#PWR084" H 1550 5550 50  0001 C CNN
+F 0 "#PWR082" H 1550 5550 50  0001 C CNN
 F 1 "+5V" H 1550 5840 50  0000 C CNN
 F 2 "" H 1550 5700 50  0000 C CNN
@@
 P 1550 6100
 AR Path="/51047C7A" Ref="#PWR084"  Part="1"
-AR Path="/5176EFAC/51047C7A" Ref="#PWR085"  Part="1"
-F 0 "#PWR085" H 1550 6100 30  0001 C CNN
+AR Path="/5176EFAC/51047C7A" Ref="#PWR083"  Part="1"
+F 0 "#PWR083" H 1550 6100 30  0001 C CNN
 F 1 "GND" H 1550 6030 30  0001 C CNN
 F 2 "" H 1550 6100 60  0001 C CNN
@@
 F 0 "K203" V 2000 5900 50  0000 C CNN
 F 1 "S3" V 2100 5900 40  0000 C CNN
-F 2 "Pin_Headers:Pin_Header_Straight_1x03" H 2050 5900 60  0001 C CNN
+F 2 "Pin_Headers:Pin_Header_Straight_1x03_Pitch2.54mm" H 2050 5900 60  0001 C CNN
 F 3 "" H 2050 5900 60  0001 C CNN
 	1    2050 5900
@@
 F 0 "K202" V 2000 5250 50  0000 C CNN
 F 1 "S2" V 2100 5250 40  0000 C CNN
-F 2 "Pin_Headers:Pin_Header_Straight_1x03" H 2050 5250 60  0001 C CNN
+F 2 "Pin_Headers:Pin_Header_Straight_1x03_Pitch2.54mm" H 2050 5250 60  0001 C CNN
 F 3 "" H 2050 5250 60  0001 C CNN
 	1    2050 5250
@@
 P 1550 5450
 AR Path="/51047C77" Ref="#PWR085"  Part="1"
-AR Path="/5176EFAC/51047C77" Ref="#PWR086"  Part="1"
-F 0 "#PWR086" H 1550 5450 30  0001 C CNN
+AR Path="/5176EFAC/51047C77" Ref="#PWR084"  Part="1"
+F 0 "#PWR084" H 1550 5450 30  0001 C CNN
 F 1 "GND" H 1550 5380 30  0001 C CNN
 F 2 "" H 1550 5450 60  0001 C CNN
@@
 $EndComp
 $Comp
-L +5V #PWR087
+L +5V #PWR085
 U 1 1 51047C76
 P 1550 5050
-F 0 "#PWR087" H 1550 4900 50  0001 C CNN
+F 0 "#PWR085" H 1550 4900 50  0001 C CNN
 F 1 "+5V" H 1550 5190 50  0000 C CNN
 F 2 "" H 1550 5050 50  0000 C CNN
@@
 SERVO1
 $Comp
-L +5V #PWR088
+L +5V #PWR086
 U 1 1 51047C09
 P 1550 4300
-F 0 "#PWR088" H 1550 4150 50  0001 C CNN
+F 0 "#PWR086" H 1550 4150 50  0001 C CNN
 F 1 "+5V" H 1550 4440 50  0000 C CNN
 F 2 "" H 1550 4300 50  0000 C CNN
@@
 P 1550 4700
 AR Path="/51047C01" Ref="#PWR088"  Part="1"
-AR Path="/5176EFAC/51047C01" Ref="#PWR089"  Part="1"
-F 0 "#PWR089" H 1550 4700 30  0001 C CNN
+AR Path="/5176EFAC/51047C01" Ref="#PWR087"  Part="1"
+F 0 "#PWR087" H 1550 4700 30  0001 C CNN
 F 1 "GND" H 1550 4630 30  0001 C CNN
 F 2 "" H 1550 4700 60  0001 C CNN
@@
 F 0 "K201" V 2000 4500 50  0000 C CNN
 F 1 "S1" V 2100 4500 40  0000 C CNN
-F 2 "Pin_Headers:Pin_Header_Straight_1x03" H 2050 4500 60  0001 C CNN
+F 2 "Pin_Headers:Pin_Header_Straight_1x03_Pitch2.54mm" H 2050 4500 60  0001 C CNN
 F 3 "" H 2050 4500 60  0001 C CNN
 	1    2050 4500
@@
 P 5250 2600
 AR Path="/51047413" Ref="#PWR089"  Part="1"
-AR Path="/5176EFAC/51047413" Ref="#PWR090"  Part="1"
-F 0 "#PWR090" H 5250 2600 30  0001 C CNN
+AR Path="/5176EFAC/51047413" Ref="#PWR088"  Part="1"
+F 0 "#PWR088" H 5250 2600 30  0001 C CNN
 F 1 "GND" H 5250 2530 30  0001 C CNN
 F 2 "" H 5250 2600 60  0001 C CNN
@@
 F 0 "P211" V 5750 2350 50  0000 C CNN
 F 1 "I2C-0" V 5850 2350 50  0000 C CNN
-F 2 "Pin_Headers:Pin_Header_Straight_1x04" H 5800 2350 60  0001 C CNN
+F 2 "Pin_Headers:Pin_Header_Straight_1x04_Pitch2.54mm" H 5800 2350 60  0001 C CNN
 F 3 "" H 5800 2350 60  0001 C CNN
 	1    5800 2350
@@
 	9400 5725 8050 5725
 $Comp
-L +5V #PWR091
+L +5V #PWR089
 U 1 1 52421C84
 P 7950 3100
-F 0 "#PWR091" H 7950 2950 50  0001 C CNN
+F 0 "#PWR089" H 7950 2950 50  0001 C CNN
 F 1 "+5V" H 7950 3240 50  0000 C CNN
 F 2 "" H 7950 3100 50  0000 C CNN
@@
 $EndComp
 $Comp
-L +V_LOGIC #PWR092
+L +V_LOGIC #PWR090
 U 1 1 52475621
 P 10250 3650
-F 0 "#PWR092" H 10250 3620 30  0001 C CNN
+F 0 "#PWR090" H 10250 3620 30  0001 C CNN
 F 1 "+V_LOGIC" H 10250 3750 30  0000 C CNN
 F 2 "" H 10250 3650 60  0001 C CNN
@@
 P 4400 6900
 AR Path="/52B23654" Ref="#PWR092"  Part="1"
-AR Path="/5176EFAC/52B23654" Ref="#PWR093"  Part="1"
-F 0 "#PWR093" H 4400 6900 30  0001 C CNN
+AR Path="/5176EFAC/52B23654" Ref="#PWR091"  Part="1"
+F 0 "#PWR091" H 4400 6900 30  0001 C CNN
 F 1 "GND" H 4400 6830 30  0001 C CNN
 F 2 "" H 4400 6900 60  0001 C CNN
@@
 Connection ~ 3650 6150
 $Comp
-L +V_LOGIC #PWR094
+L +V_LOGIC #PWR092
 U 1 1 52B2384C
 P 4400 5600
-F 0 "#PWR094" H 4400 5570 30  0001 C CNN
+F 0 "#PWR092" H 4400 5570 30  0001 C CNN
 F 1 "+V_LOGIC" H 4400 5700 30  0000 C CNN
 F 2 "" H 4400 5600 60  0001 C CNN
@@
 P 6050 6600
 AR Path="/52B22346" Ref="#PWR094"  Part="1"
-AR Path="/5176EFAC/52B22346" Ref="#PWR095"  Part="1"
-F 0 "#PWR095" H 6050 6600 30  0001 C CNN
+AR Path="/5176EFAC/52B22346" Ref="#PWR093"  Part="1"
+F 0 "#PWR093" H 6050 6600 30  0001 C CNN
 F 1 "GND" H 6050 6530 30  0001 C CNN
 F 2 "" H 6050 6600 60  0001 C CNN
@@
 	6050 6400 6050 6600
 $Comp
-L +V_LOGIC #PWR096
+L +V_LOGIC #PWR094
 U 1 1 52B2234D
 P 6050 5900
-F 0 "#PWR096" H 6050 5870 30  0001 C CNN
+F 0 "#PWR094" H 6050 5870 30  0001 C CNN
 F 1 "+V_LOGIC" H 6050 6000 30  0000 C CNN
 F 2 "" H 6050 5900 60  0001 C CNN
