File: RAMPS-FD/con_outputs.sch (KiCad schematic (older format))
At the start: 24 parts, among them P218 D11, P403 D9, P404 D8, P405 D10, Q201 IRLB8743PBF, Q202 IRLB8743PBF, Q203 IRLB8743PBF, Q206 IRLB8743PBF

Commit message: Changed fuse holders to Keystone 3568; specificy HCT instead of ACT logic
Parts:
- D201, D202, D203, D204: symbol LED -> LED-RESCUE-RAMPS-FD
- D401, D402, D403, D404: symbol DIODE -> D
Connections:
- net +V_HEATBED: now also D404.1 (K); no longer D404.2 (K)
- net +V_POWER: now also D401.1 (K), D402.1 (K), D403.1 (K); no longer D401.2 (K), D402.2 (K), D403.2 (K)
- net D10_OUT: now also D402.2 (A); no longer D402.1 (A)
- net D8_OUT: now also D404.2 (A); no longer D404.1 (A)
- net D9_OUT: now also D401.2 (A); no longer D401.1 (A)
- net FET4_OUT: now also D403.2 (A); no longer D403.1 (A)
Changed lines of the file:
@@
 	9800 5200 10250 5200
 Wire Wire Line
-	9450 5050 9450 5450
+	9450 5000 9450 5450
 Wire Wire Line
 	2850 5350 4350 5350
@@
 Connection ~ 3650 2050
 Wire Wire Line
-	3650 2050 3650 1700
+	3650 2050 3650 1650
 Connection ~ 9600 1950
 Wire Wire Line
-	9600 1950 9600 1600
+	9600 1950 9600 1550
 Wire Wire Line
 	4500 1850 4100 1850
@@
 	10000 1750 10000 850
 Wire Wire Line
-	9600 650  9600 1200
+	9600 650  9600 1250
 Connection ~ 3650 850
 Wire Wire Line
-	3350 5000 3350 5500
+	3350 4950 3350 5500
 Wire Wire Line
 	2700 2050 4500 2050
@@
 	2700 2050 2700 2000
 Wire Wire Line
-	3650 700  3650 1300
+	3650 700  3650 1350
 Wire Wire Line
 	4350 5150 3750 5150
@@
 	3750 5150 3750 4300
 Wire Wire Line
-	9450 4050 9450 4650
+	9450 4050 9450 4700
 Wire Wire Line
 	9000 5400 10250 5400
@@
 	2000 5800 3050 5800
 Wire Wire Line
-	3350 4150 3350 4600
+	3350 4150 3350 4650
 Text Notes 6750 1800 0    80   ~ 0
 FET4 - Extruder 3 / Fan
@@
 $EndComp
 $Comp
-L DIODE D404
+L D D404
 U 1 1 51A9D334
 P 3650 1500
@@
 F 3 "" H 3650 1500 60  0001 C CNN
 	1    3650 1500
-	0    -1   -1   0
-$EndComp
-$Comp
-L DIODE D403
+	0    1    1    0
+$EndComp
+$Comp
+L D D403
 U 1 1 519E92CD
 P 9600 1400
@@
 F 3 "" H 9600 1400 60  0001 C CNN
 	1    9600 1400
-	0    -1   -1   0
-$EndComp
-$Comp
-L DIODE D401
+	0    1    1    0
+$EndComp
+$Comp
+L D D401
 U 1 1 519E9216
 P 3350 4800
@@
 F 3 "" H 3350 4800 60  0001 C CNN
 	1    3350 4800
-	0    -1   -1   0
-$EndComp
-$Comp
-L DIODE D402
+	0    1    1    0
+$EndComp
+$Comp
+L D D402
 U 1 1 5186017E
 P 9450 4850
@@
 F 3 "" H 9450 4850 60  0001 C CNN
 	1    9450 4850
-	0    -1   -1   0
+	0    1    1    0
 $EndComp
 $Comp
@@
 $EndComp
 $Comp
-L LED D204
+L LED-RESCUE-RAMPS-FD D204
 U 1 1 51770EF9
 P 8900 1700
@@
 MOSFET Outputs
 $Comp
-L LED D203
+L LED-RESCUE-RAMPS-FD D203
 U 1 1 51047AB7
 P 2850 5100
@@
 $EndComp
 $Comp
-L LED D202
+L LED-RESCUE-RAMPS-FD D202
 U 1 1 510479AE
 P 9000 5150
@@
 $EndComp
 $Comp
-L LED D201
+L LED-RESCUE-RAMPS-FD D201
 U 1 1 510478C6
 P 2700 1800
