File: RAMPS-FD/e-stop.sch (KiCad schematic (older format))
At the start: 17 parts, among them P302 ESTOP, Q1 DMN2075, U1 74ACT125, U2 74ACT244

Commit message: Changed fuse holders to Keystone 3568; specificy HCT instead of ACT logic
Parts:
- D1: symbol LED -> LED-RESCUE-RAMPS-FD
- D301: footprint w_smd_diode:SOD323 -> Diodes_SMD:SOD-123; symbol DIODE -> D
- U1: value 74ACT125 -> 74HCT125
- U2: value 74ACT244 -> 74HCT244
Connections:
- net ESTOP: now also D301.1 (K); no longer D301.2 (K)
- net at P302.1 (P1), Q1.G, R304.2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: now also D301.2 (A); no longer D301.1 (A)
Other:
- note added: "Must use HCT type buffers. \nInputs are compatible with \n3.3V or 5V logic"
- note removed: "Must use ACT (or HCT) type buffers. \nInputs are compatible with \n3.3V or 5V logic"
Changed lines of the file:
@@
 P 4850 6450
 F 0 "U1" H 4850 6550 50  0000 L BNN
-F 1 "74ACT125" H 4900 6300 40  0000 L TNN
+F 1 "74HCT125" H 4900 6300 40  0000 L TNN
 F 2 "Housings_SSOP:TSSOP-14_4.4x5mm_Pitch0.65mm" H 4850 6450 60  0001 C CNN
 F 3 "" H 4850 6450 60  0001 C CNN
@@
 P 4900 5700
 F 0 "U1" H 4900 5800 50  0000 L BNN
-F 1 "74ACT125" H 4950 5550 40  0000 L TNN
+F 1 "74HCT125" H 4950 5550 40  0000 L TNN
 F 2 "Housings_SSOP:TSSOP-14_4.4x5mm_Pitch0.65mm" H 4900 5700 60  0001 C CNN
 F 3 "" H 4900 5700 60  0001 C CNN
@@
 P 4900 5100
 F 0 "U1" H 4900 5200 50  0000 L BNN
-F 1 "74ACT125" H 4950 4950 40  0000 L TNN
+F 1 "74HCT125" H 4950 4950 40  0000 L TNN
 F 2 "Housings_SSOP:TSSOP-14_4.4x5mm_Pitch0.65mm" H 4900 5100 60  0001 C CNN
 F 3 "" H 4900 5100 60  0001 C CNN
@@
 P 4900 4350
 F 0 "U1" H 4900 4450 50  0000 L BNN
-F 1 "74ACT125" H 4950 4200 40  0000 L TNN
+F 1 "74HCT125" H 4950 4200 40  0000 L TNN
 F 2 "Housings_SSOP:TSSOP-14_4.4x5mm_Pitch0.65mm" H 4900 4350 60  0001 C CNN
 F 3 "" H 4900 4350 60  0001 C CNN
@@
 P 5100 2800
 F 0 "U2" H 5150 2600 60  0000 C CNN
-F 1 "74ACT244" H 5200 2400 60  0000 C CNN
+F 1 "74HCT244" H 5200 2400 60  0000 C CNN
 F 2 "Housings_SSOP:TSSOP-20_4.4x6.5mm_Pitch0.65mm" H 5100 2800 60  0001 C CNN
 F 3 "" H 5100 2800 60  0001 C CNN
@@
 D8
 $Comp
-L DIODE D301
+L D D301
 U 1 1 51B65AB0
 P 1900 1600
 F 0 "D301" H 1900 1700 40  0000 C CNN
 F 1 "1N4148" H 1900 1500 40  0000 C CNN
-F 2 "w_smd_diode:SOD323" H 1900 1600 60  0001 C CNN
+F 2 "Diodes_SMD:SOD-123" H 1900 1600 60  0001 C CNN
 F 3 "" H 1900 1600 60  0001 C CNN
 	1    1900 1600
-	1    0    0    1
+	-1   0    0    -1
 $EndComp
 $Comp
@@
 VCC = 5V
 Text Notes 9500 2950 0    60   ~ 12
-Must use ACT (or HCT) type buffers. \nInputs are compatible with \n3.3V or 5V logic
+Must use HCT type buffers. \nInputs are compatible with \n3.3V or 5V logic
 Wire Wire Line
 	5350 5100 7650 5100
@@
 	10100 900  10100 1150
 Wire Wire Line
-	2100 1600 2500 1600
+	2050 1600 2500 1600
 Wire Wire Line
 	5800 2700 7600 2700
@@
 	1300 2350 1300 2200
 Wire Wire Line
-	1150 1600 1700 1600
+	1150 1600 1750 1600
 Wire Wire Line
 	5800 2900 7600 2900
@@
 	825  1450 825  775
 $Comp
-L LED D1
+L LED-RESCUE-RAMPS-FD D1
 U 1 1 5725588E
 P 1450 4850
