File: RAMPS-FD/steppers2.sch (KiCad schematic (older format))
At the start: 15 parts, among them P207 3 2 1, P208 3 2 1, P209 3 2 1, P210 E2, P212 E1, P217 E0, U204 E2, U205 E1, U206 E0

Commit message: Changed fuse holders to Keystone 3568; specificy HCT instead of ACT logic
Parts:
- P207, P208, P209: footprint pin_array:pin_array_3x2 -> Pin_Headers:Pin_Header_Straight_2x03
Changed lines of the file:
@@
 F 0 "P209" H 3000 4650 50  0000 C CNN
 F 1 "3 2 1" V 3000 4450 40  0000 C CNN
-F 2 "pin_array:pin_array_3x2" H 3000 4400 60  0001 C CNN
+F 2 "Pin_Headers:Pin_Header_Straight_2x03" H 3000 4400 60  0001 C CNN
 F 3 "" H 3000 4400 60  0001 C CNN
 	1    3000 4400
@@
 F 0 "P208" H 3000 2250 50  0000 C CNN
 F 1 "3 2 1" V 3000 2050 40  0000 C CNN
-F 2 "pin_array:pin_array_3x2" H 3000 2000 60  0001 C CNN
+F 2 "Pin_Headers:Pin_Header_Straight_2x03" H 3000 2000 60  0001 C CNN
 F 3 "" H 3000 2000 60  0001 C CNN
 	1    3000 2000
@@
 F 0 "P207" H 2900 7100 50  0000 C CNN
 F 1 "3 2 1" V 2900 6900 40  0000 C CNN
-F 2 "pin_array:pin_array_3x2" H 2900 6850 60  0001 C CNN
+F 2 "Pin_Headers:Pin_Header_Straight_2x03" H 2900 6850 60  0001 C CNN
 F 3 "" H 2900 6850 60  0001 C CNN
 	1    2900 6850

Commit message: Fix 3d view; remove faulty ADC protection
Parts:
- C204, C205, C206: footprint Capacitors_SMD:c_elec_6.3x7.7 -> Capacitors_SMD:CP_Elec_6.3x7.7
- P207, P208, P209: footprint Pin_Headers:Pin_Header_Straight_2x03 -> Pin_Headers:Pin_Header_Straight_2x03_Pitch2.54mm
Changed lines of the file:
@@
 F 0 "P209" H 3000 4650 50  0000 C CNN
 F 1 "3 2 1" V 3000 4450 40  0000 C CNN
-F 2 "Pin_Headers:Pin_Header_Straight_2x03" H 3000 4400 60  0001 C CNN
+F 2 "Pin_Headers:Pin_Header_Straight_2x03_Pitch2.54mm" H 3000 4400 60  0001 C CNN
 F 3 "" H 3000 4400 60  0001 C CNN
 	1    3000 4400
@@
 P 5600 5250
 AR Path="/51B4E8DF" Ref="#PWR059"  Part="1"
-AR Path="/51B4E84F/51B4E8DF" Ref="#PWR060"  Part="1"
-F 0 "#PWR060" H 5600 5250 30  0001 C CNN
+AR Path="/51B4E84F/51B4E8DF" Ref="#PWR058"  Part="1"
+F 0 "#PWR058" H 5600 5250 30  0001 C CNN
 F 1 "GND" H 5600 5180 30  0001 C CNN
 F 2 "" H 5600 5250 60  0001 C CNN
@@
 P 5700 2800
 AR Path="/51B4E8DC" Ref="#PWR060"  Part="1"
-AR Path="/51B4E84F/51B4E8DC" Ref="#PWR061"  Part="1"
-F 0 "#PWR061" H 5700 2800 30  0001 C CNN
+AR Path="/51B4E84F/51B4E8DC" Ref="#PWR059"  Part="1"
+F 0 "#PWR059" H 5700 2800 30  0001 C CNN
 F 1 "GND" H 5700 2730 30  0001 C CNN
 F 2 "" H 5700 2800 60  0001 C CNN
@@
 F 0 "P208" H 3000 2250 50  0000 C CNN
 F 1 "3 2 1" V 3000 2050 40  0000 C CNN
-F 2 "Pin_Headers:Pin_Header_Straight_2x03" H 3000 2000 60  0001 C CNN
+F 2 "Pin_Headers:Pin_Header_Straight_2x03_Pitch2.54mm" H 3000 2000 60  0001 C CNN
 F 3 "" H 3000 2000 60  0001 C CNN
 	1    3000 2000
@@
 F 0 "C206" H 6350 1900 50  0000 L CNN
 F 1 "100u 35V" H 6350 1700 50  0000 L CNN
-F 2 "Capacitors_SMD:c_elec_6.3x7.7" H 6300 1800 60  0001 C CNN
+F 2 "Capacitors_SMD:CP_Elec_6.3x7.7" H 6300 1800 60  0001 C CNN
 F 3 "" H 6300 1800 60  0001 C CNN
 	1    6300 1800
@@
 F 0 "C205" H 6250 4300 50  0000 L CNN
 F 1 "100u 35V" H 6250 4100 50  0000 L CNN
-F 2 "Capacitors_SMD:c_elec_6.3x7.7" H 6200 4200 60  0001 C CNN
+F 2 "Capacitors_SMD:CP_Elec_6.3x7.7" H 6200 4200 60  0001 C CNN
 F 3 "" H 6200 4200 60  0001 C CNN
 	1    6200 4200
@@
 F 0 "C204" H 6150 6750 50  0000 L CNN
 F 1 "100u 35V" H 6150 6550 50  0000 L CNN
-F 2 "Capacitors_SMD:c_elec_6.3x7.7" H 6100 6650 60  0001 C CNN
+F 2 "Capacitors_SMD:CP_Elec_6.3x7.7" H 6100 6650 60  0001 C CNN
 F 3 "" H 6100 6650 60  0001 C CNN
 	1    6100 6650
@@
 P 5500 7700
 AR Path="/51B4E8CF" Ref="#PWR061"  Part="1"
-AR Path="/51B4E84F/51B4E8CF" Ref="#PWR062"  Part="1"
-F 0 "#PWR062" H 5500 7700 30  0001 C CNN
+AR Path="/51B4E84F/51B4E8CF" Ref="#PWR060"  Part="1"
+F 0 "#PWR060" H 5500 7700 30  0001 C CNN
 F 1 "GND" H 5500 7630 30  0001 C CNN
 F 2 "" H 5500 7700 60  0001 C CNN
@@
 F 0 "P207" H 2900 7100 50  0000 C CNN
 F 1 "3 2 1" V 2900 6900 40  0000 C CNN
-F 2 "Pin_Headers:Pin_Header_Straight_2x03" H 2900 6850 60  0001 C CNN
+F 2 "Pin_Headers:Pin_Header_Straight_2x03_Pitch2.54mm" H 2900 6850 60  0001 C CNN
 F 3 "" H 2900 6850 60  0001 C CNN
 	1    2900 6850
@@
 $EndComp
 $Comp
-L +V_MOTOR #PWR063
+L +V_MOTOR #PWR061
 U 1 1 51B4E8CC
 P 5450 6000
-F 0 "#PWR063" H 5450 5970 30  0001 C CNN
+F 0 "#PWR061" H 5450 5970 30  0001 C CNN
 F 1 "+V_MOTOR" H 5450 6100 30  0000 C CNN
 F 2 "" H 5450 6000 60  0001 C CNN
@@
 $EndComp
 $Comp
-L +V_MOTOR #PWR064
+L +V_MOTOR #PWR062
 U 1 1 51B4E8CB
 P 5550 3550
-F 0 "#PWR064" H 5550 3520 30  0001 C CNN
+F 0 "#PWR062" H 5550 3520 30  0001 C CNN
 F 1 "+V_MOTOR" H 5550 3650 30  0000 C CNN
 F 2 "" H 5550 3550 60  0001 C CNN
@@
 $EndComp
 $Comp
-L +V_MOTOR #PWR065
+L +V_MOTOR #PWR063
 U 1 1 51B4E8CA
 P 5650 1150
-F 0 "#PWR065" H 5650 1120 30  0001 C CNN
+F 0 "#PWR063" H 5650 1120 30  0001 C CNN
 F 1 "+V_MOTOR" H 5650 1250 30  0000 C CNN
 F 2 "" H 5650 1150 60  0001 C CNN
@@
 $EndComp
 $Comp
-L +V_LOGIC #PWR066
+L +V_LOGIC #PWR064
 U 1 1 51B4E8C9
 P 3550 5550
-F 0 "#PWR066" H 3550 5520 30  0001 C CNN
+F 0 "#PWR064" H 3550 5520 30  0001 C CNN
 F 1 "+V_LOGIC" H 3550 5650 30  0000 C CNN
 F 2 "" H 3550 5550 60  0001 C CNN
@@
 $EndComp
 $Comp
-L +V_LOGIC #PWR067
+L +V_LOGIC #PWR065
 U 1 1 51B4E8C8
 P 3650 3100
-F 0 "#PWR067" H 3650 3070 30  0001 C CNN
+F 0 "#PWR065" H 3650 3070 30  0001 C CNN
 F 1 "+V_LOGIC" H 3650 3200 30  0000 C CNN
 F 2 "" H 3650 3100 60  0001 C CNN
@@
 $EndComp
 $Comp
-L +V_LOGIC #PWR068
+L +V_LOGIC #PWR066
 U 1 1 51B4E8C7
 P 3750 700
-F 0 "#PWR068" H 3750 670 30  0001 C CNN
+F 0 "#PWR066" H 3750 670 30  0001 C CNN
 F 1 "+V_LOGIC" H 3750 800 30  0000 C CNN
 F 2 "" H 3750 700 60  0001 C CNN
@@
 $EndComp
 $Comp
-L +V_LOGIC #PWR069
+L +V_LOGIC #PWR067
 U 1 1 51B4E8C6
 P 3800 2250
-F 0 "#PWR069" H 3800 2220 30  0001 C CNN
+F 0 "#PWR067" H 3800 2220 30  0001 C CNN
 F 1 "+V_LOGIC" H 3800 2350 30  0000 C CNN
 F 2 "" H 3800 2250 60  0001 C CNN
@@
 $EndComp
 $Comp
-L +V_LOGIC #PWR070
+L +V_LOGIC #PWR068
 U 1 1 51B4E8C5
 P 3600 7100
-F 0 "#PWR070" H 3600 7070 30  0001 C CNN
+F 0 "#PWR068" H 3600 7070 30  0001 C CNN
 F 1 "+V_LOGIC" H 3600 7200 30  0000 C CNN
 F 2 "" H 3600 7100 60  0001 C CNN
@@
 $EndComp
 $Comp
-L +V_LOGIC #PWR071
+L +V_LOGIC #PWR069
 U 1 1 51B4E8C4
 P 3700 4650
-F 0 "#PWR071" H 3700 4620 30  0001 C CNN
+F 0 "#PWR069" H 3700 4620 30  0001 C CNN
 F 1 "+V_LOGIC" H 3700 4750 30  0000 C CNN
 F 2 "" H 3700 4650 60  0001 C CNN
